File: SEGmeter25.sch (EAGLE design)
At the start: 133 parts, among them IC1 DS1307, IC2 LD1117S50, IC3 LD1117S33, IC4 XBEE, IC5 ATmega328, IC6 MCP1541, IC7 MCP3208, J1 Short 12V, J10 3.5mm, J11 3.5mm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

Commit message: foo
Other:
- note added: "V2.5 (03-07-2012)"
- note removed: "V0.5 (03-07-2012)"
Changed lines of the file:
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@@
 <wire x1="312.166" y1="17.78" x2="312.166" y2="12.7" width="0.3048" layer="94"/>
 <text x="259.08" y="20.32" size="3.048" layer="94">Smart Energy Groups SEGmeter v2.5</text>
-<text x="284.48" y="14.478" size="1.778" layer="94">V0.5 (03-07-2012)</text>
+<text x="284.48" y="14.478" size="1.778" layer="94">V2.5 (03-07-2012)</text>
 <text x="259.08" y="14.478" size="1.778" layer="94">foo</text>
 <text x="258.826" y="9.398" size="1.778" layer="94">(C)2012 Luke Weston</text>
@@
 <wire x1="101.346" y1="17.78" x2="101.346" y2="12.7" width="0.3048" layer="94"/>
 <text x="48.26" y="20.32" size="3.048" layer="94">Smart Energy Groups SEGmeter v2.5</text>
-<text x="73.66" y="14.478" size="1.778" layer="94">V0.5 (03-07-2012)</text>
+<text x="73.66" y="14.478" size="1.778" layer="94">V2.5 (03-07-2012)</text>
 <text x="48.26" y="14.478" size="1.778" layer="94">foo</text>
 <text x="48.006" y="9.398" size="1.778" layer="94">(C)2012 Luke Weston</text>
@@
 <wire x1="446.786" y1="360.68" x2="446.786" y2="355.6" width="0.3048" layer="94"/>
 <text x="393.7" y="363.22" size="3.048" layer="94">Smart Energy Groups SEGmeter v2.5</text>
-<text x="419.1" y="357.378" size="1.778" layer="94">V0.5 (03-07-2012)</text>
+<text x="419.1" y="357.378" size="1.778" layer="94">V2.5 (03-07-2012)</text>
 <text x="393.7" y="357.378" size="1.778" layer="94">foo</text>
 <text x="393.446" y="352.298" size="1.778" layer="94">(C)2012 Luke Weston</text>
@@
 <wire x1="60.706" y1="205.74" x2="60.706" y2="200.66" width="0.3048" layer="94"/>
 <text x="7.62" y="208.28" size="3.048" layer="94">Smart Energy Groups SEGmeter v2.5</text>
-<text x="33.02" y="202.438" size="1.778" layer="94">V0.5 (03-07-2012)</text>
+<text x="33.02" y="202.438" size="1.778" layer="94">V2.5 (03-07-2012)</text>
 <text x="7.62" y="202.438" size="1.778" layer="94">foo</text>
 <text x="7.366" y="197.358" size="1.778" layer="94">(C)2012 Luke Weston</text>
