File: SEGmeter25.sch (EAGLE design)
At the start: 133 parts, among them IC1 DS1307, IC2 LD1117S50, IC3 LD1117S33, IC4 XBEE, IC5 ATmega328, IC6 MCP1541, IC7 MCP3208, J1 Short 12V, J10 3.5mm, J11 3.5mm, J12 Relays, J13 3.5mm, J14 Star ground, J15 3.5mm, J16 Arduino-compatible headers, J17 3.5mm, J18 3.5mm, J2 1-Wire, J3 ISP, J4 Power, J5 Comms, J6 MICROSD, J7 Sensor 5V, J8 3.5mm, J9 3.5mm, Q1 32768 Hz, Q2 16 MHz, Q3 2N7002, Q4 2N7002, Q5 2N7002

Commit message: foo
Parts:
- removed JP5, JP6, JP7: FIDUCIAL1.5X3, SparkFun:FIDUCIAL1.5X3
- added D4: 1N4148, SparkFun:DIODESOD
- added FID1, FID2, FID3: FIDUCIAL, adafruit:FIDUCIAL
- added J19, J20: 3.5mm, SparkFun:AUDIO-JACKSMD2
- J12: value Relays -> 3.5mm; device con-phoenix-254:MPT6 -> SparkFun:AUDIO-JACKSMD2
- J14: value Star ground -> Relays; device freetronics-luke:SJ -> con-phoenix-254:MPT6
- J16: value Arduino-compatible headers -> Star ground; device Arduino-Various:ARDUINO-USBNO-OUTLINE-NO-TEXT-OCTAGONAL -> freetronics-luke:SJ
- J18: value 3.5mm -> Arduino-compatible headers; device SparkFun:AUDIO-JACKSMD2 -> Arduino-Various:ARDUINO-USBNO-OUTLINE-NO-TEXT-OCTAGONAL
- J7: value Sensor 5V -> Buttons; device freetronics-luke:SJ -> con-phoenix-254:MPT6
- J8: value 3.5mm -> Relay LEDs; device SparkFun:AUDIO-JACKSMD2 -> con-phoenix-254:MPT6
- J9: value 3.5mm -> Sensor 5V; device SparkFun:AUDIO-JACKSMD2 -> freetronics-luke:SJ
- LED1: value Status -> RSSI
- LED2: value Power -> Assoc
- LED3: value RSSI -> Status
- LED4: value Assoc -> Power
- R1, R2: value 1k -> 4k7
- R11, R17, R7, R8: value 10k -> 1k
- R12: value 3k3 -> 1k
- R13, R14, R9: value 1k -> 10k
- R15: value 10k -> 220k
- R16: value 2k2 -> 3k3
- R21: value 220k -> 1k
- R22: value 1k -> 2k2
- R30, R31: value 3k3 -> 220k
- R33, R34: value 220k -> 3k3
- R5, R6: value 4k7 -> 10k
- renumbered JP1 to H1, JP2 to H2, JP3 to H3, JP4 to H4
Connections:
- removed net N$24: LED5.A, R30.1
- removed net N$25: R12.2, S2.1
- removed net N$27: LED6.A, R31.1
- removed net N$31: R12.1, R13.2, S3.1
- removed net N$58: LED7.A, R32.1
- removed net N$72: D1.C, D2.C, D3.C, J12-1.1, J12-3.1, J12-5.1, R30.2, R31.2, R32.2, SJ1.2
- new net BUTTON1: J7-2.1, R16.2, S2.1
- new net BUTTON2: J7-4.1, R16.1, R19.2, S3.1
- new net N$3: D1.A, J5.10, J5.9
- new net RELAY1LED: J8-2.1, LED5.C, R32.2
- new net RELAY2LED: J8-4.1, LED6.C, R33.2
- new net RELAY3LED: J8-6.1, LED7.C, R34.2
- new net RELAY_VOLTAGE: D2.C, D3.C, D4.C, J14-1.1, J14-3.1, J14-5.1, J8-1.1, J8-3.1, J8-5.1, LED5.A, LED6.A, LED7.A, SJ1.2
- net !ADC1_CS: now also J18.10_PWM; no longer J16.10_PWM
- net !ADC2_CS: now also J18.9_PWM; no longer J16.9_PWM
- net !GPIO_CS: now also R9.1; no longer R11.1
- net !RESET: now also J18.RESET, R5.2; no longer J16.RESET, R7.2
- net +12V: now also D1.C, J18.VIN; no longer J16.VIN
- net +3V3: now also J18.3V3, R9.2; no longer J16.3V3, R11.2
- net +5V: now also J18.5V, J7-1.1, J7-3.1, J7-5.1, J9.2, R1.2, R12.2, R5.1; no longer J16.5V, J7.2, R4.2, R5.2, R7.1
- net 1WIRE: now also J18.5_PWM, R3.1; no longer J16.5_PWM, R5.1
- net 3.3VTXD: now also R4.2, R6.1; no longer R6.2, R8.1
- net A1: now also J18.A_1; no longer J16.A_1
- net A2: now also J18.A_2; no longer J16.A_2
- net A3: now also J18.A_3; no longer J16.A_3
- net AGND: now also J12.SLEEVE, J16.2, J19.SLEEVE, J20.SLEEVE, R18.1, R30.1; no longer J14.2, J18.SLEEVE, J8.SLEEVE, J9.SLEEVE, R20.1, R33.1
- net AREF: now also J18.AREF; no longer J16.AREF
- net BUTTONS: now also J18.A_0, J7-6.1, R19.1, R22.2; no longer J16.A_0, R13.1, R16.2
- net GND: now also J16.1, J18.GND0, J18.GND1, J18.GND2, R14.2, R22.1, R6.2; no longer J14.1, J16.GND0, J16.GND1, J16.GND2, R16.1, R17.2, R8.2
- net MISO: now also J18.12; no longer J16.12
- net MOSI: now also J18.11_PWM; no longer J16.11_PWM
- net N$1: now also LED4.A, R12.1; no longer LED2.A, R2.1
- net N$18: now also D2.A, J14-2.1, R32.1; no longer D1.A, J12-2.1, LED5.C
- net N$2: now also LED3.A, R11.1; no longer LED1.A, R1.1
- net N$26: now also D3.A, J14-4.1, R33.1; no longer D2.A, J12-4.1, LED6.C
- net N$30: now also J20.LEFT; no longer J18.LEFT
- net N$4: now also R7.1; no longer R9.1
- net N$40: now also D4.A, J14-6.1, R34.1; no longer D3.A, J12-6.1, LED7.C
- net N$41: now also J19.LEFT; no longer J17.LEFT
- net N$42: now also J10.LEFT; no longer J8.LEFT
- net N$44: now also J11.LEFT; no longer J9.LEFT
- net N$45: now also J17.LEFT; no longer J15.LEFT
- net N$46: now also J12.RIGHT, J19.RIGHT, J20.RIGHT, J9.1; no longer J18.RIGHT, J7.1, J8.RIGHT, J9.RIGHT
- net N$47: now also J15.LEFT; no longer J13.LEFT
- net N$48: now also J13.LEFT; no longer J11.LEFT
- net N$49: now also J12.LEFT; no longer J10.LEFT
- net N$5: now also R8.1; no longer R10.1
- net N$50: now also R15.1, R17.2, R18.2; no longer R18.1, R19.2, R20.2
- net N$54: now also R31.1; no longer R34.1
- net N$55: now also R20.1, R21.2; no longer R21.1, R22.2
- net N$57: now also R30.2; no longer R33.2
- net N$6: now also LED2.A, R8.2; no longer LED4.A, R10.2
- net N$60: now also R21.1; no longer R22.1
- net N$7: now also LED1.A, R7.2; no longer LED3.A, R9.2
- net N$70: now also R17.1; no longer R19.1
- net RELAY1: now also J18.6_PWM; no longer J16.6_PWM
- net RELAY2: now also J18.7; no longer J16.7
- net RELAY3: now also J18.8; no longer J16.8
- net RXD: now also J18.0_RX, R10.2; no longer J16.0_RX, R14.2
- net SCK: now also J18.13; no longer J16.13
- net SCL: now also J18.A_5, R1.1; no longer J16.A_5, R3.1
- net SDA: now also J18.A_4, R2.1; no longer J16.A_4, R4.1
- net SIN: now also R13.1, R14.1; no longer R15.1, R17.1
- net SOUT: now also R10.1; no longer R14.1
- net SPARE: now also J18.2; no longer J16.2
- net SPARE2: now also J18.4; no longer J16.4
- net STATUS_LED: now also J18.3_PWM, R11.2; no longer J16.3_PWM, R1.2
- net TXD: now also J18.1_TX, R13.2, R4.1; no longer J16.1_TX, R15.2, R6.1
- net V+: now also R15.2, R20.2, R31.2; no longer R18.2, R21.2, R34.2
Other:
- moved on the sheet: D1, D2, D3, J10, J11, J13, J15, J17, J2-1, J2-2, J2-3, LED1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

Commit message: foo
Parts:
- C5, C6: value 27pF -> 22pF
- Q1: device SparkFun:CRYSTALTC26H -> SparkFun:CRYSTAL32-SMD
- Q2: value 16 MHz -> 16MHz; device freetronics-master-v1:CRYSTALHC49US -> SparkFun:CRYSTAL5X3
- R11, R12: value 1k -> 330R
- R32, R33, R34: value 3k3 -> 1k
Connections:
- net N$28: now also Q2.1; no longer Q2.2
- net N$29: now also Q2.2; no longer Q2.1
Other:
- note added: "5x3.2mm"
- note added: "CTX820CT-ND"
- note removed: "HC49US"
- moved on the sheet: Q2
Changed lines of the file:
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@@
 <part name="R5" library="freetronics-master-v1" deviceset="RESISTOR" device="0805" value="10k"/>
 <part name="P+3" library="supply1" deviceset="+5V" device=""/>
-<part name="Q2" library="freetronics-master-v1" deviceset="CRYSTAL" device="HC49US" value="16 MHz"/>
-<part name="C6" library="freetronics-master-v1" deviceset="CAP" device="0805" value="27pF"/>
-<part name="C5" library="freetronics-master-v1" deviceset="CAP" device="0805" value="27pF"/>
+<part name="C6" library="freetronics-master-v1" deviceset="CAP" device="0805" value="22pF"/>
+<part name="C5" library="freetronics-master-v1" deviceset="CAP" device="0805" value="22pF"/>
 <part name="P+4" library="supply1" deviceset="+5V" device=""/>
 <part name="U$21" library="freetronics-luke" deviceset="GND" device=""/>
@@
 <part name="P+7" library="supply1" deviceset="+12V" device=""/>
 <part name="LED4" library="freetronics-master-v1" deviceset="LED" device="0805" value="Power"/>
-<part name="R12" library="freetronics-master-v1" deviceset="RESISTOR" device="0805" value="1k"/>
+<part name="R12" library="freetronics-master-v1" deviceset="RESISTOR" device="0805" value="330R"/>
 <part name="U$29" library="freetronics-luke" deviceset="GND" device=""/>
 <part name="P+9" library="supply1" deviceset="+5V" device=""/>
 <part name="LED3" library="freetronics-master-v1" deviceset="LED" device="0805" value="Status"/>
-<part name="R11" library="freetronics-master-v1" deviceset="RESISTOR" device="0805" value="1k"/>
+<part name="R11" library="freetronics-master-v1" deviceset="RESISTOR" device="0805" value="330R"/>
 <part name="U$30" library="freetronics-luke" deviceset="GND" device=""/>
 <part name="J10" library="SparkFun" deviceset="AUDIO-JACK" device="SMD2" value="3.5mm"/>
@@
 <part name="U$56" library="freetronics-luke" deviceset="+5V" device=""/>
 <part name="B1" library="SparkFun" deviceset="BATTERY" device="12MM" value="CR1220"/>
-<part name="Q1" library="SparkFun" deviceset="CRYSTAL" device="TC26H" value="32768 Hz"/>
 <part name="C3" library="freetronics-master-v1" deviceset="CAP" device="0805" value="100nF"/>
 <part name="U$59" library="freetronics-luke" deviceset="GND" device=""/>
@@
 <part name="J8" library="con-phoenix-254" deviceset="MPT6" device="" value="Relay LEDs"/>
 <part name="U$58" library="freetronics-luke" deviceset="+5V" device=""/>
-<part name="R32" library="freetronics-master-v1" deviceset="RESISTOR" device="0805" value="3k3"/>
-<part name="R33" library="freetronics-master-v1" deviceset="RESISTOR" device="0805" value="3k3"/>
-<part name="R34" library="freetronics-master-v1" deviceset="RESISTOR" device="0805" value="3k3"/>
+<part name="R32" library="freetronics-master-v1" deviceset="RESISTOR" device="0805" value="1k"/>
+<part name="R33" library="freetronics-master-v1" deviceset="RESISTOR" device="0805" value="1k"/>
+<part name="R34" library="freetronics-master-v1" deviceset="RESISTOR" device="0805" value="1k"/>
 <part name="R16" library="freetronics-master-v1" deviceset="RESISTOR" device="0805" value="3k3"/>
 <part name="R19" library="freetronics-master-v1" deviceset="RESISTOR" device="0805" value="1k"/>
@@
 <part name="D1" library="SparkFun" deviceset="DIODE" device="SOD" value="1N4148"/>
 <part name="P+11" library="supply1" deviceset="+12V" device=""/>
+<part name="Q2" library="SparkFun" deviceset="CRYSTAL" device="5X3" value="16MHz"/>
+<part name="Q1" library="SparkFun" deviceset="CRYSTAL" device="32-SMD" value="32768 Hz"/>
 </parts>
 <sheets>
@@
 <text x="22.86" y="276.86" size="1.27" layer="98">0805</text>
 <text x="33.02" y="256.54" size="1.27" layer="98">0805</text>
-<text x="33.02" y="276.86" size="1.27" layer="98">HC49US</text>
 <text x="35.56" y="236.22" size="1.27" layer="98">0805</text>
 <text x="22.86" y="233.68" size="1.27" layer="98">0805</text>
@@
 <text x="269.24" y="124.46" size="1.27" layer="98">0805</text>
 <text x="172.72" y="266.7" size="1.27" layer="98">SOD-323</text>
+<text x="33.02" y="276.86" size="1.27" layer="98">5x3.2mm</text>
+<text x="30.48" y="279.4" size="1.27" layer="98">CTX820CT-ND</text>
 </plain>
 <instances>
@@
 </instance>
 <instance part="P+3" gate="1" x="38.1" y="302.26" smashed="yes" rot="MR0">
-<attribute name="VALUE" x="33.02" y="299.72" size="1.27" layer="96"/>
-</instance>
-<instance part="Q2" gate="G$1" x="35.56" y="266.7" smashed="yes" rot="R90">
-<attribute name="NAME" x="33.02" y="274.32" size="1.27" layer="95"/>
-<attribute name="VALUE" x="33.02" y="271.78" size="1.27" layer="96"/>
+<attribute name="VALUE" x="40.64" y="299.72" size="1.27" layer="96"/>
 </instance>
 <instance part="C6" gate="G$1" x="27.94" y="264.16" smashed="yes" rot="R270">
@@
 <attribute name="VALUE" x="165.1" y="322.58" size="1.27" layer="96"/>
 </instance>
-<instance part="Q1" gate="G$1" x="160.02" y="337.82" smashed="yes">
-<attribute name="NAME" x="154.94" y="342.9" size="1.27" layer="95"/>
-<attribute name="VALUE" x="154.94" y="340.868" size="1.27" layer="96"/>
-</instance>
 <instance part="C3" gate="G$1" x="190.5" y="327.66" smashed="yes" rot="R180">
 <attribute name="NAME" x="195.58" y="325.12" size="1.27" layer="95"/>
@@
 <instance part="P+11" gate="1" x="180.34" y="274.32" smashed="yes" rot="R270">
 <attribute name="VALUE" x="177.546" y="276.86" size="1.27" layer="96"/>
+</instance>
+<instance part="Q2" gate="G$1" x="35.56" y="266.7" smashed="yes" rot="R270">
+<attribute name="NAME" x="33.02" y="274.32" size="1.27" layer="95"/>
+<attribute name="VALUE" x="33.02" y="271.78" size="1.27" layer="96"/>
+</instance>
+<instance part="Q1" gate="G$1" x="160.02" y="337.82" smashed="yes">
+<attribute name="NAME" x="154.94" y="342.9" size="1.27" layer="95"/>
+<attribute name="VALUE" x="154.94" y="340.868" size="1.27" layer="96"/>
 </instance>
 </instances>
@@
 <wire x1="40.64" y1="269.24" x2="35.56" y2="269.24" width="0.1524" layer="91"/>
 <pinref part="IC5" gate="1" pin="PB6(XTAL1/TOSC1/PCINT6)"/>
-<pinref part="Q2" gate="G$1" pin="2"/>
+<pinref part="C5" gate="G$1" pin="1"/>
+<pinref part="Q2" gate="G$1" pin="1"/>
 <wire x1="35.56" y1="269.24" x2="33.02" y2="269.24" width="0.1524" layer="91"/>
 <junction x="35.56" y="269.24"/>
-<pinref part="C5" gate="G$1" pin="1"/>
 </segment>
 </net>
@@
 <wire x1="40.64" y1="264.16" x2="35.56" y2="264.16" width="0.1524" layer="91"/>
 <pinref part="IC5" gate="1" pin="PB7(XTAL2/TOSC2/PCINT7)"/>
-<pinref part="Q2" gate="G$1" pin="1"/>
+<pinref part="C6" gate="G$1" pin="1"/>
+<pinref part="Q2" gate="G$1" pin="2"/>
 <wire x1="35.56" y1="264.16" x2="33.02" y2="264.16" width="0.1524" layer="91"/>
 <junction x="35.56" y="264.16"/>
-<pinref part="C6" gate="G$1" pin="1"/>
 </segment>
 </net>
@@
 </segment>
 </net>
-<net name="N$10" class="0">
-<segment>
-<pinref part="IC1" gate="G$1" pin="X2"/>
-<pinref part="Q1" gate="G$1" pin="2"/>
-<wire x1="162.56" y1="337.82" x2="165.1" y2="337.82" width="0.1524" layer="91"/>
-</segment>
-</net>
 <net name="N$12" class="0">
 <segment>
-<pinref part="Q1" gate="G$1" pin="1"/>
-<wire x1="157.48" y1="337.82" x2="154.94" y2="337.82" width="0.1524" layer="91"/>
 <wire x1="154.94" y1="337.82" x2="154.94" y2="340.36" width="0.1524" layer="91"/>
 <pinref part="IC1" gate="G$1" pin="X1"/>
 <wire x1="154.94" y1="340.36" x2="165.1" y2="340.36" width="0.1524" layer="91"/>
+<wire x1="154.94" y1="337.82" x2="157.48" y2="337.82" width="0.1524" layer="91"/>
+<pinref part="Q1" gate="G$1" pin="1"/>
 </segment>
 </net>
@@
 </segment>
 </net>
+<net name="N$8" class="0">
+<segment>
+<pinref part="IC1" gate="G$1" pin="X2"/>
+<wire x1="162.56" y1="337.82" x2="165.1" y2="337.82" width="0.1524" layer="91"/>
+<pinref part="Q1" gate="G$1" pin="2"/>
+</segment>
+</net>

Commit message: foo
Parts:
- R7, R8: value 1k -> 330R
Changed lines of the file:
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@@
 <part name="IC4" library="Luke" deviceset="XBEE" device=""/>
 <part name="IC3" library="burr-brown" deviceset="REG1117" device="" value="LD1117S33"/>
-<part name="R7" library="freetronics-master-v1" deviceset="RESISTOR" device="0805" value="1k"/>
+<part name="R7" library="freetronics-master-v1" deviceset="RESISTOR" device="0805" value="330R"/>
 <part name="C7" library="freetronics-master-v1" deviceset="CAP" device="0805" value="10uF"/>
 <part name="LED1" library="freetronics-master-v1" deviceset="LED" device="0805" value="RSSI"/>
@@
 <part name="U$46" library="freetronics-luke" deviceset="+3.3V" device=""/>
 <part name="LED2" library="freetronics-master-v1" deviceset="LED" device="0805" value="Assoc"/>
-<part name="R8" library="freetronics-master-v1" deviceset="RESISTOR" device="0805" value="1k"/>
+<part name="R8" library="freetronics-master-v1" deviceset="RESISTOR" device="0805" value="330R"/>
 <part name="R6" library="freetronics-master-v1" deviceset="RESISTOR" device="0805" value="10k"/>
 <part name="R4" library="freetronics-master-v1" deviceset="RESISTOR" device="0805" value="4k7"/>
