File: SEGmeter25.brd (EAGLE design)
At the start: 114.3 x 87.6 mm, 137 parts, among them IC1 DS1307, IC2 LD1117S50, IC3 LD1117S33, IC4 XBEE, IC5 ATmega328, IC6 MCP1541, IC7 MCP3208, J1 Short 12V, J10 3.5mm, J11 3.5mm, J12 3.5mm, J13 3.5mm, J14 Relays, J15 3.5mm, J16 Star ground, J17 3.5mm, J18 Arduino-compatible headers, J19 3.5mm, J2 1-Wire, J20 3.5mm, J3 ISP, J4 Power, J5 Comms, J6 MICROSD, J7 Buttons, J8 Relay LEDs, J9 Sensor 5V, Q1 32768 Hz, Q2 16 MHz, Q3 2N7002, Q4 2N7002, Q5 2N7002

Commit message: foo
Routing:
- net RELAY2: track 77.0 -> 78.9 mm
Changed lines of the file:
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@@
 <wire x1="47.625" y1="39.37" x2="46.99" y2="38.735" width="0.4064" layer="1"/>
 <wire x1="24.4475" y1="50.43" x2="24.8175" y2="50.43" width="0.4064" layer="1"/>
-<wire x1="46.99" y1="38.735" x2="38.735" y2="38.735" width="0.4064" layer="1"/>
+<wire x1="46.99" y1="38.735" x2="35.56" y2="38.735" width="0.4064" layer="1"/>
 <wire x1="24.4475" y1="50.43" x2="33.39" y2="50.43" width="0.4064" layer="1"/>
 <wire x1="33.39" y1="50.43" x2="34.29" y2="49.53" width="0.4064" layer="1"/>
-<wire x1="34.29" y1="49.53" x2="34.29" y2="43.18" width="0.4064" layer="1"/>
-<wire x1="34.29" y1="43.18" x2="38.735" y2="38.735" width="0.4064" layer="1"/>
+<wire x1="34.29" y1="49.53" x2="34.29" y2="40.005" width="0.4064" layer="1"/>
+<wire x1="34.29" y1="40.005" x2="35.56" y2="38.735" width="0.4064" layer="1"/>
 </signal>
 <signal name="RELAY3">
@@
 <wire x1="59.055" y1="46.99" x2="58.42" y2="46.355" width="0.4064" layer="1"/>
 <via x="58.42" y="46.355" extent="1-16" drill="0.4"/>
-<wire x1="58.42" y1="46.355" x2="52.705" y2="46.355" width="0.4064" layer="16"/>
-<via x="52.705" y="46.355" extent="1-16" drill="0.4"/>
+<wire x1="58.42" y1="46.355" x2="52.07" y2="46.355" width="0.4064" layer="16"/>
+<via x="52.07" y="46.355" extent="1-16" drill="0.4"/>
 <wire x1="19.7104" y1="65.4304" x2="19.7104" y2="63.95085" width="0.4064" layer="1"/>
 <wire x1="19.7104" y1="63.95085" x2="20.193" y2="63.46825" width="0.4064" layer="1"/>
@@
 <wire x1="48.8425" y1="45.905625" x2="48.26" y2="45.323125" width="0.4064" layer="1"/>
 <wire x1="48.26" y1="45.323125" x2="48.26" y2="43.815" width="0.4064" layer="1"/>
-<wire x1="52.705" y1="46.355" x2="50.8" y2="46.355" width="0.4064" layer="1"/>
+<wire x1="52.07" y1="46.355" x2="50.8" y2="46.355" width="0.4064" layer="1"/>
 <wire x1="50.8" y1="46.355" x2="50.165" y2="46.99" width="0.4064" layer="1"/>
 <wire x1="50.165" y1="46.99" x2="48.8425" y2="46.99" width="0.4064" layer="1"/>

Commit message: foo
Parts:
- moved H1 28.8 mm to (-1.27, 1.59)
- moved H4 24.7 mm to (105.4, 1.91)
- moved H2 4.84 mm to (-1.27, 81.9)
- moved H3 4.26 mm to (105.4, 81.9)
- moved J4 1.42 mm to (94.0, 34.9), turned to 270 degrees
- moved FID2 1.27 mm to (0.00, 6.99)
Routing:
- net +12V: track 184.8 -> 205.3 mm
Changed lines of the file:
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@@
 <setting verticaltext="up"/>
 </settings>
-<grid distance="25" unitdist="mil" unit="mil" style="lines" multiple="1" display="yes" altdistance="6.25" altunitdist="mil" altunit="mil"/>
+<grid distance="50" unitdist="mil" unit="mil" style="lines" multiple="1" display="yes" altdistance="12.5" altunitdist="mil" altunit="mil"/>
 <layers>
 <layer number="1" name="Top" color="4" fill="1" visible="yes" active="yes"/>
@@
 <text x="38.1" y="46.99" size="0.8128" layer="21" ratio="15">GND/</text>
 <text x="38.1" y="45.72" size="0.8128" layer="21" ratio="15">AGND</text>
-<text x="85.09" y="28.575" size="0.8128" layer="21" ratio="15">(7-12V DC 500mA-1A)</text>
+<text x="87.63" y="40.005" size="0.8128" layer="21" ratio="15">(7-12V DC 500mA-1A)</text>
 <dimension x1="-5.08" y1="80.01" x2="109.22" y2="80.01" x3="52.07" y3="85.725" layer="48"/>
 <wire x1="104.775" y1="40.64" x2="102.87" y2="38.735" width="0" layer="20" curve="90"/>
@@
 </autorouter>
 <elements>
-<element name="H4" library="SparkFun" package="STAND-OFF" value="STAND-OFF" x="100.33" y="26.035" smashed="yes" rot="R180"/>
+<element name="H4" library="SparkFun" package="STAND-OFF" value="STAND-OFF" x="105.41" y="1.905" smashed="yes" rot="R180"/>
 <element name="IC5" library="avr-5" package="DIL28-3" value="ATmega328" x="50.8" y="58.42" smashed="yes">
 <attribute name="VALUE" x="32.385" y="52.07" size="0.762" layer="27" ratio="12"/>
@@
 <element name="U$1" library="OSHW" package="OSHW_8X200_NOTEXT" value="" x="15.24" y="28.575" smashed="yes"/>
 <element name="J6" library="adafruit" package="MICROSD" value="MICROSD" x="86.36" y="55.88" smashed="yes" rot="R90"/>
-<element name="H3" library="SparkFun" package="STAND-OFF" value="STAND-OFF" x="101.6" y="80.01" smashed="yes"/>
-<element name="H2" library="SparkFun" package="STAND-OFF" value="STAND-OFF" x="3.175" y="80.01" smashed="yes"/>
-<element name="H1" library="SparkFun" package="STAND-OFF" value="STAND-OFF" x="13.97" y="26.035" smashed="yes"/>
+<element name="H3" library="SparkFun" package="STAND-OFF" value="STAND-OFF" x="105.41" y="81.915" smashed="yes"/>
+<element name="H2" library="SparkFun" package="STAND-OFF" value="STAND-OFF" x="-1.27" y="81.915" smashed="yes"/>
+<element name="H1" library="SparkFun" package="STAND-OFF" value="STAND-OFF" x="-1.27" y="1.5875" smashed="yes"/>
 <element name="J5" library="pinhead" package="2X06" value="Comms" x="89.535" y="79.375" smashed="yes"/>
 <element name="S1" library="SparkFun" package="TACTILE_SWITCH_SMD" value="Reset" x="44.45" y="79.375" smashed="yes" rot="R180"/>
@@
 <attribute name="VALUE" x="72.80275" y="71.9455" size="0.762" layer="27" ratio="12"/>
 </element>
-<element name="J4" library="SparkFun" package="POWER_JACK_SLOT" value="Power" x="92.71" y="34.29" smashed="yes" rot="R90">
-<attribute name="VALUE" x="88.265" y="40.64" size="0.8128" layer="27" ratio="15"/>
+<element name="J4" library="SparkFun" package="POWER_JACK_SLOT" value="Power" x="93.98" y="34.925" smashed="yes" rot="R270">
+<attribute name="VALUE" x="88.9" y="41.275" size="0.8128" layer="27" ratio="15"/>
 </element>
 <element name="IC2" library="burr-brown" package="SOT223" value="LD1117S50" x="19.685" y="68.58" smashed="yes">
@@
 </element>
 <element name="FID1" library="adafruit" package="FIDUCIAL_1MM" value="FIDUCIAL" x="80.645" y="57.229375"/>
-<element name="FID2" library="adafruit" package="FIDUCIAL_1MM" value="FIDUCIAL" x="0" y="5.715"/>
+<element name="FID2" library="adafruit" package="FIDUCIAL_1MM" value="FIDUCIAL" x="0" y="6.985"/>
 <element name="FID3" library="adafruit" package="FIDUCIAL_1MM" value="FIDUCIAL" x="0.635" y="64.135"/>
 <element name="J7" library="con-phoenix-254" package="6POL254" value="Buttons" x="3.81" y="50.8" smashed="yes" rot="R90">
@@
 <wire x1="93.1475" y1="54.530625" x2="79.295625" y2="54.530625" width="0.6096" layer="1"/>
 <wire x1="79.295625" y1="54.530625" x2="76.835" y2="52.07" width="0.6096" layer="1"/>
-<wire x1="86.614" y1="34.29" x2="86.614" y2="42.291" width="0.4064" layer="16"/>
-<wire x1="86.614" y1="42.291" x2="76.835" y2="52.07" width="0.4064" layer="16"/>
+<wire x1="79.375" y1="49.53" x2="76.835" y2="52.07" width="0.4064" layer="16"/>
+<wire x1="100.076" y1="34.925" x2="97.79" y2="34.925" width="0.4064" layer="16"/>
+<wire x1="97.79" y1="34.925" x2="94.615" y2="31.75" width="0.4064" layer="16"/>
+<wire x1="94.615" y1="31.75" x2="92.075" y2="31.75" width="0.4064" layer="16"/>
+<wire x1="92.075" y1="31.75" x2="91.44" y2="32.385" width="0.4064" layer="16"/>
+<wire x1="91.44" y1="32.385" x2="91.44" y2="48.26" width="0.4064" layer="16"/>
+<wire x1="91.44" y1="48.26" x2="90.17" y2="49.53" width="0.4064" layer="16"/>
+<wire x1="90.17" y1="49.53" x2="79.375" y2="49.53" width="0.4064" layer="16"/>
 </signal>
 <signal name="RELAY1">
@@
 <wire x1="101.6" y1="47.36" x2="101.6" y2="44.715" width="0.4064" layer="1"/>
 <contactref element="R22" pad="1"/>
-<wire x1="92.71" y1="34.29" x2="92.71" y2="47.625" width="0.4064" layer="16"/>
+<wire x1="93.98" y1="34.925" x2="94.615" y2="34.925" width="0.4064" layer="16"/>
+<wire x1="94.615" y1="34.925" x2="94.615" y2="47.625" width="0.4064" layer="16"/>
 </signal>
 <signal name="BUTTON2">

Commit message: foo
Parts:
- C5, C6: value 27pF -> 22pF
- Q1: device SparkFun:TC26H -> SparkFun:CRYSTAL-32KHZ-SMD
- Q2: value 16 MHz -> 16MHz; device freetronics-master-v1:HC49US -> SparkFun:CRYSTAL-SMD-5X3
- R11, R12: value 1k -> 330R
- R32, R33, R34: value 3k3 -> 1k
- turned Q2 to 0 degrees
Connections:
- removed net N$10: IC1.2, Q1.2
- new net N$8: IC1.2, Q1.X2
- net N$12: now also Q1.X1; no longer Q1.1
- net N$28: now also Q2.1; no longer Q2.2
- net N$29: now also Q2.3; no longer Q2.1
Routing:
- net N$10: track 6.69 -> 0.00 mm
- net N$8: track 0.00 -> 6.50 mm
- net N$28: track 10.2 -> 13.3 mm
- net RELAY1: track 75.6 -> 74.1 mm
- net +12V: track 205.3 -> 204.1 mm
- net MISO: track 64.3 -> 63.2 mm, vias 1 -> 2
- net +5V: track 338.1 -> 337.6 mm, vias 14 -> 12
- net SCK: vias 0 -> 1
Other:
- board text added: "SmartEnergyGroups.com"
- board text added: "This fine Internet of Things device was crafted with"
- board text added: "email sam@smartenergygroups.com"
- board text added: "love by @lukeweston and @samotage to help everybody"
- board text added: "on up to our internets website or"
- board text added: "save electrons everywhere. If you would like to know"
- board text added: "some more about this device, roll"

Commit message: foo
Parts:
- R7, R8: value 1k -> 330R
Changed lines of the file:
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@@
 <attribute name="VALUE" x="24.511" y="73.05675" size="0.762" layer="27" ratio="12"/>
 </element>
-<element name="R7" library="freetronics-master-v1" package="0805" value="1k" x="101.6" y="52.07" smashed="yes" rot="R270">
-<attribute name="VALUE" x="99.6315" y="50.83175" size="0.762" layer="27" ratio="12"/>
+<element name="R7" library="freetronics-master-v1" package="0805" value="330R" x="101.6" y="52.07" smashed="yes" rot="R270">
+<attribute name="VALUE" x="98.044" y="50.19675" size="0.762" layer="27" ratio="12"/>
 </element>
 <element name="C7" library="freetronics-master-v1" package="0805" value="10uF" x="27.305" y="62.865" smashed="yes">
@@
 <attribute name="VALUE" x="102.9065" y="42.5655" size="0.762" layer="27" ratio="12" rot="SR0"/>
 </element>
-<element name="R8" library="freetronics-master-v1" package="0805" value="1k" x="99.06" y="43.815" smashed="yes" rot="R270">
-<attribute name="VALUE" x="97.0915" y="42.57675" size="0.762" layer="27" ratio="12"/>
+<element name="R8" library="freetronics-master-v1" package="0805" value="330R" x="99.06" y="43.815" smashed="yes" rot="R270">
+<attribute name="VALUE" x="95.504" y="43.21175" size="0.762" layer="27" ratio="12"/>
 </element>
 <element name="R6" library="freetronics-master-v1" package="0805" value="10k" x="78.74" y="66.675" smashed="yes" rot="R270">
